Commit message: added inverse kinematics for 3DOF control

File: a1_description/xacro/const.xacro (robot description, xacro)
@@ -31,6 +31,6 @@
     <xacro:property name="damping" value="0"/>
     <xacro:property name="friction" value="0"/>
-    <xacro:property name="hip_max" value="0"/>   <!-- wie ein affe hab ich das auf 0 gesetzt man-->
-    <xacro:property name="hip_min" value="0"/>
+    <xacro:property name="hip_max" value="46"/>   <!-- wie ein affe hab ich das auf 0 gesetzt man-->
+    <xacro:property name="hip_min" value="-46"/>
     <xacro:property name="hip_velocity_max" value="21"/>
     <xacro:property name="hip_torque_max" value="33.5"/>
